Commit message: 'DummyVecEnv works as serial env with dartEnv'

File: DartEnv2/gym/envs/dart/assets/KR5/ground.urdf (robot description, URDF)
Before this commit: robot ground_skeleton, 2 links, 1 joints
Links:
- link ground_link: geometry collision box size=4.0 0.05 4.0; visual box size=4.0 0.05 4.0
