Commit message: "simulation failure management"

File: DartEnv2/gym/envs/dart/assets/KR5/KR5 sixx R650 ball.urdf (robot description, URDF)
Before this commit: robot KR5sixxR650WP_description, 8 links, 7 joints
Links:
- link base_link: geometry visual mesh filename=meshes/base_link.STL
- link bicep: geometry visual mesh filename=meshes/bicep.STL
- link elbow: geometry visual mesh filename=meshes/elbow.STL
- link forearm: geometry visual mesh filename=meshes/forearm.STL
- link shoulder: geometry visual mesh filename=meshes/shoulder.STL
