Commit message: 'added iiwa arm support'

File: DartEnv2/gym/envs/dart/assets/kuka_lbr_iiwa_support/lbr_iiwa_14_r820.urdf (robot description, URDF)
Before this commit: robot kuka_lbr_iiwa_14_r820, 11 links, 10 joints
Links:
- link base_link: geometry visual mesh filename=meshes/lbr_iiwa_14_r820/visual/base_link.stl
- link link_1: geometry visual mesh filename=meshes/lbr_iiwa_14_r820/visual/link_1.stl
- link link_2: geometry visual mesh filename=meshes/lbr_iiwa_14_r820/visual/link_2.stl
- link link_3: geometry visual mesh filename=meshes/lbr_iiwa_14_r820/visual/link_3.stl
- link link_4: geometry visual mesh filename=meshes/lbr_iiwa_14_r820/visual/link_4.stl
- link link_5: geometry visual mesh filename=meshes/lbr_iiwa_14_r820/visual/link_5.stl
- link link_6: geometry visual mesh filename=meshes/lbr_iiwa_14_r820/visual/link_6.stl
